File: STM32 - BLDC Driver/untitled.kicad_sch (KiCad schematic)
At the start: 15 parts, among them J1 Conn_01x02_Pin, U2 LM2596S-3.3, U7 LM66100DCK

Commit message: Started assigning footprints
Parts:
- removed R39: 5Ohm, symbol Device:R
- added R44: 5kOhm (C2073749), Resistor_SMD:R_0805_2012Metric_Pad1.20x1.40mm_HandSolder, symbol Device:R
- C1: value C - Low ESR Electrolytic -> 680uF LOW ESR ( C443017 ); footprint (none) -> Capacitor_THT:C_Radial_D12.5mm_H20.0mm_P5.00mm
- C2: value 0.1uF Ceramic -> 0.1uF Ceramic (CL21B104KBCNNNC ); footprint (none) -> Capacitor_SMD:C_0805_2012Metric
- C3: value TPSC337K006R0080 -> C600568; footprint (none) -> Capacitor_Tantalum_SMD:CP_EIA-7343-43_Kemet-X
- D1: value SR502 -> SR502 (HandSoldered); footprint (none) -> Diode_THT:D_DO-27_P12.70mm_Horizontal
- D2: footprint (none) -> LED_SMD:LED_0805_2012Metric_Pad1.15x1.40mm_HandSolder
- J1: footprint (none) -> Connector_AMASS:AMASS_XT30PW-M_1x02_P2.50mm_Horizontal
- L1: value PE-54040 -> 7447720330 (HandSolder); footprint (none) -> Inductor_THT:L_Radial_D7.8mm_P5.00mm_Fastron_07HCP
- R1: value 5Ohm -> 5Ohm (C17724); footprint (none) -> Resistor_SMD:R_0805_2012Metric_Pad1.20x1.40mm_HandSolder
Connections:
- net +3V3: now also R44.1
- net at U7.5 (ST): now also R44.2
Other:
- moved on the sheet: C1
