File: STM32 - BLDC Driver/untitled.kicad_sch (KiCad schematic)
At the start: 15 parts, among them J1 Conn_01x02_Pin, U2 LM2596S-3.3, U7 LM66100DCK

Commit message: As manufactured.
Parts:
- removed C1: 680uF LOW ESR ( C443017 ), Capacitor_THT:C_Radial_D12.5mm_H20.0mm_P5.00mm, symbol Device:C
- removed C2: 0.1uF Ceramic (CL21B104KBCNNNC ), Capacitor_SMD:C_0805_2012Metric, symbol Device:C
- removed C3: C600568, Capacitor_Tantalum_SMD:CP_EIA-7343-43_Kemet-X, symbol Device:C
- removed D1: SR502 (HandSoldered), Diode_THT:D_DO-27_P12.70mm_Horizontal, symbol Device:D
- removed D2: C2297, LED_SMD:LED_0805_2012Metric_Pad1.15x1.40mm_HandSolder, symbol Device:LED
- removed L1: 7447720330 (HandSolder), Inductor_THT:L_Radial_D7.8mm_P5.00mm_Fastron_07HCP, symbol Device:L
- removed R1: 5Ohm (C17724), Resistor_SMD:R_0805_2012Metric_Pad1.20x1.40mm_HandSolder, symbol Device:R
- removed R44: 5kOhm (C2073749), Resistor_SMD:R_0805_2012Metric_Pad1.20x1.40mm_HandSolder, symbol Device:R
- removed TP1, TP3, TP4: TestPoint, symbol Connector:TestPoint
- removed U2: LM2596S-3.3, Package_TO_SOT_SMD:TO-263-5_TabPin3, symbol Regulator_Switching:LM2596S-3.3
- added C36, C37, C38, C39, C40, C75: 22uF (C45783), Capacitor_SMD:C_0805_2012Metric_Pad1.18x1.45mm_HandSolder, symbol Device:C
- added C41: 100uF 63V (C7471891), Capacitor_SMD:C_Elec_8x10.2, symbol Device:C
- added C42, C43: 4.7u low esr (C1779), Capacitor_SMD:C_0805_2012Metric_Pad1.18x1.45mm_HandSolder, symbol Device:C
- added C44, C67: 4.7uF 50V (C29823), Capacitor_SMD:C_1206_3216Metric_Pad1.33x1.80mm_HandSolder, symbol Device:C
- added C45, C66: 100nF 50V (C28233), Capacitor_SMD:C_0805_2012Metric_Pad1.18x1.45mm_HandSolder, symbol Device:C
- added C68, C74: 0.1uF (C28233), Capacitor_SMD:C_0805_2012Metric_Pad1.18x1.45mm_HandSolder, symbol Device:C
- added L2, L4: 15uH (C216196), Inductor_SMD:L_7.3x7.3_H3.5, symbol Device:L
- added R59, R62: 64.9k (C17788), Resistor_SMD:R_0805_2012Metric_Pad1.20x1.40mm_HandSolder, symbol Device:R
- added R60: 100k (C15458), Resistor_SMD:R_0603_1608Metric_Pad0.98x0.95mm_HandSolder, symbol Device:R
- added R61, R64: 24.9k (C17571), Resistor_SMD:R_0805_2012Metric_Pad1.20x1.40mm_HandSolder, symbol Device:R
- added R63: 57.6k (C204216), Resistor_SMD:R_0603_1608Metric_Pad0.98x0.95mm_HandSolder, symbol Device:R
- added TP12: TestPoint, TestPoint:TestPoint_Pad_D4.0mm, symbol Connector:TestPoint
- added U1, U3: LMR38020SDDAR, DDA0008E-IPC_A, symbol 2025-09-26_20-56-39:LMR38020SDDAR
- added U6: LM66100DCK, Package_TO_SOT_SMD:SOT-363_SC-70-6, symbol Power_Management:LM66100DCK
- TP11: renamed from TP2; footprint (none) -> TestPoint:TestPoint_Pad_D4.0mm
- renumbered J1 to J9
Connections:
- net +3V3: now also C42.1, C43.1, U6.6 (VOUT); no longer U7.3 (~{CE})
- net GND: now also C36.1, C37.1, C38.1, C39.1, C40.1, C41.1, C42.2, C43.2, C44.2, C45.1, C66.1, C67.2, C75.1, R59.2, R61.2, R62.2, R64.2, U1.1 (PGND), U1.9 (EP), U3.1 (PGND), U3.9 (EP), U6.2 (GND)
- net MAIN_3V3: now reaches U7.1 (VIN)
- net MAIN_3V3: now also C36.2, C37.2, C75.2, L2.2, R63.1, U6.3 (~{CE})
- net +24V renamed PVDD
- net PVDD: now also C41.2, C44.1, C45.2, C66.2, C67.1, TP12.1, U1.2 (EN), U1.3 (VIN), U3.2 (EN), U3.3 (VIN)
- new net: R59.1, U3.4 (RT_SYNC)
- new net: R63.2, R64.1, U3.5 (FB)
- new net: C74.1, U3.7 (BOOT)
- new net: C74.2, L2.1, U3.8 (SW)
- new net: R62.1, U1.4 (RT_SYNC)
- new net: R60.2, R61.1, U1.5 (FB)
- new net: C68.1, U1.7 (BOOT)
- new net: C68.2, L4.1, U1.8 (SW)
- new net 5V: C38.2, C39.2, C40.2, L4.2, R60.1
- new net USB_3V3: U6.1 (VIN), U7.3 (~{CE})
- no-connect marks 0 -> 4
Other:
- note added: "3V3"
- note added: "5V"
- note removed: "Switching regulator 24V to 3V3 3A Check and verify before ordering: C,L,D"
- note removed: "This should prevent reverse current"
