File: STM32 - BLDC Driver/STM32 - BLDC Driver.kicad_pcb (KiCad board)
At the start: 2 copper layers, 6 parts, among them J4 TC2050, U1 STM32F411CEUx, U2 LM2596S-3.3, U6 LD1117S33TR_SOT223, U7 LM66100DCK, U8 LM66100DCK

Commit message: Footprints
Parts:
- added C1: 680uF LOW ESR ( C443017 ), Capacitor_THT:C_Radial_D12.5mm_H20.0mm_P5.00mm, F.Cu at (108.8, 40.5)
- added C2: 0.1uF Ceramic (CL21B104KBCNNNC ), Capacitor_SMD:C_0805_2012Metric, F.Cu at (116.4, 49.1)
- added C3: C600568, Capacitor_Tantalum_SMD:CP_EIA-7343-43_Kemet-X, F.Cu at (109.3, 50.5)
- added D1: SR502 (HandSoldered), Diode_THT:D_DO-27_P12.70mm_Horizontal, F.Cu at (106.3, 30.1)
- added D2: C2297, LED_SMD:LED_0805_2012Metric_Pad1.15x1.40mm_HandSolder, F.Cu at (101.1, 51.0)
- added J1: Conn_01x02_Pin, Connector_AMASS:AMASS_XT30PW-M_1x02_P2.50mm_Horizontal, F.Cu at (99.1, 40.8)
- added L1: 7447720330 (HandSolder), Inductor_THT:L_Radial_D7.8mm_P5.00mm_Fastron_07HCP, F.Cu at (91.3, 48.4)
- added R1: 5Ohm (C17724), Resistor_SMD:R_0805_2012Metric_Pad1.20x1.40mm_HandSolder, F.Cu at (101.1, 45.0)
- added R44: 5kOhm (C2073749), Resistor_SMD:R_0805_2012Metric_Pad1.20x1.40mm_HandSolder, F.Cu at (101.1, 48.0)
