File: STM32 - BLDC Driver/BLDC MOSFETS.kicad_sch (KiCad schematic)
At the start: 49 parts, among them Q1 Q_NMOS_Depletion_SGD, Q2 Q_NMOS_Depletion_SGD, Q3 Q_NMOS_Depletion_SGD, Q4 Q_NMOS_Depletion_SGD, Q5 Q_NMOS_Depletion_SGD, Q6 Q_NMOS_Depletion_SGD, U4 AS5600

Commit message: As manufactured.
Parts:
- removed C32: 100nF, symbol Device:C
- removed C38, C40, C42: 2.2uF, symbol Device:C
- removed C39, C41, C43: 0.1uF, symbol Device:C
- removed C49: 1000pf, symbol Device:C
- removed D6, D7: D_Zener, symbol Device:D_Zener
- removed Q1, Q2, Q3, Q4, Q5, Q6: Q_NMOS_Depletion_SGD, symbol Transistor_FET_Other:Q_NMOS_Depletion_SGD
- removed R17: DNP, symbol Device:R
- removed R22, R31: 34.8k, symbol Device:R
- removed R23, R28, R32: 4.99k, symbol Device:R
- removed R24, R25, R26, R29, R30: 10R, symbol Device:R
- removed TP10, TP11, TP12, TP13, TP14, TP17, TP18, TP5, TP6, TP8, TP9: TestPoint, symbol Connector:TestPoint
- removed U4: AS5600, AS5600:SOIC8, symbol AS5600:AS5600
- added C51, C61, C62: 0.1uF (C28233), Capacitor_SMD:C_0805_2012Metric_Pad1.18x1.45mm_HandSolder, symbol Device:C
- added C55, C59, C60: 2.2uF (C50254), Capacitor_SMD:C_1206_3216Metric_Pad1.33x1.80mm_HandSolder, symbol Device:C
- added C56: 1nF (C9196), Capacitor_SMD:C_1206_3216Metric_Pad1.33x1.80mm_HandSolder, symbol Device:C
- added D5, D8: D_Zener (C67528), Diode_SMD:D_SOD-323, symbol Device:D_Zener
- added J10: Screw_Terminal_01x03, TerminalBlock:TerminalBlock_bornier-3_P5.08mm, symbol Connector:Screw_Terminal_01x03
- added NT2, NT3, NT4, NT6, NT8: NetTie_2, NetTie:NetTie-2_SMD_Pad0.5mm, symbol Device:NetTie_2
- added Q1, Q2, Q3, Q4, Q5, Q6: SIR182DP-T1-RE3, SIR182DP:TRANS_SIR182DP-T1-RE3, symbol SIR182DP-T1-RE3:SIR182DP-T1-RE3
- added R42: 10mOhm (C393072), Resistor_SMD:R_2512_6332Metric_Pad1.40x3.35mm_HandSolder, symbol Device:R
- added R43, R50: 34.8k (C23141), Resistor_SMD:R_0603_1608Metric_Pad0.98x0.95mm_HandSolder, symbol Device:R
- added R44, R49, R51, R53, R56: 10R (C17415), Resistor_SMD:R_0805_2012Metric_Pad1.20x1.40mm_HandSolder, symbol Device:R
- added R47, R48: 4.99k (C23046), Resistor_SMD:R_0603_1608Metric_Pad0.98x0.95mm_HandSolder, symbol Device:R
- added TP20, TP21, TP24, TP25, TP26: TestPoint, TestPoint:TestPoint_Pad_D3.0mm, symbol Connector:TestPoint
- C53: renamed from C48; value 1000pf -> 1nF (C9196); footprint (none) -> Capacitor_SMD:C_1206_3216Metric
- D7: renamed from D8; value D_Zener -> D_Zener (C67528); footprint (none) -> Diode_SMD:D_SOD-323
- R45: value 10mOhm -> 4.99k (C23046); footprint (none) -> Resistor_SMD:R_0603_1608Metric_Pad0.98x0.95mm_HandSolder
- R46: renamed from R21; value 10R -> 10R (C17415); footprint (none) -> Resistor_SMD:R_0805_2012Metric_Pad1.20x1.40mm_HandSolder
- R52: renamed from R27; value 34.8k -> 34.8k (C23141); footprint (none) -> Resistor_SMD:R_0603_1608Metric_Pad0.98x0.95mm_HandSolder
- R55: renamed from R46; value 10mOhm -> 10mOhm (C393072); footprint (none) -> Resistor_SMD:R_2512_6332Metric_Pad1.40x3.35mm_HandSolder
- TP15, TP16, TP19: footprint (none) -> TestPoint:TestPoint_Pad_D3.0mm
- TP23: renamed from TP7; footprint (none) -> TestPoint:TestPoint_Pad_D3.0mm
Connections:
- net MOT_PHASE_C is gone; now on net GL_A: TP19.1
- net ASENSE: now also R45.2, TP15.1, C51.2, D5.2 (A), R43.1
- net BSENSE: now also C62.2, D8.2 (A), R48.2
- net CSENSE: now also C61.2, R47.2, R50.1, TP25.1
- net GH_A: now also TP16.1
- net GH_B: now also R49.1, TP26.1
- net GH_C: now also R53.1, TP20.1
- net GL_A: now also R44.2
- net GL_B: now also R51.1, TP24.1
- net GL_C: now also R56.1, TP21.1
- net GND: now also R45.1, C51.1, C61.1, C62.1, R47.1, R48.1
- net PGND: now also C55.2, C56.1, C59.2, C60.2, NT2.1, NT3.2, NT4.2, Q3.1, Q3.2, Q3.3, R42.1; no longer R45.1
- net PVDD: now also C55.1, C59.1, C60.1, Q2.5, Q2.6, Q2.7, Q2.8, Q2.9, Q4.5, Q4.6, Q4.7, Q4.8, Q4.9, Q5.5, Q5.6, Q5.7, Q5.8, Q5.9
- net SL_A: now also NT8.2, Q1.1, Q1.2, Q1.3, R42.2; no longer R45.2, TP16.1
- net SL_B: now also C56.2, NT6.2, Q6.1, Q6.2, Q6.3
- net VCC: now also D5.1 (K), D8.1 (K)
- net at R46.2: now also Q2.4
- net MOT_PHASE_B renamed SH_B
- net SH_B: now also J10.2 (Pin_2), Q4.1, Q4.2, Q4.3, Q6.5, Q6.6, Q6.7, Q6.8, Q6.9; no longer TP15.1
- new net: Q3.4, R56.2
- new net: Q4.4, R49.2
- new net: Q6.4, R51.2
- new net: Q5.4, R53.2
- new net: Q1.4, R44.1
- new net SH_A: J10.3 (Pin_3), Q1.5, Q1.6, Q1.7, Q1.8, Q1.9, Q2.1, Q2.2, Q2.3, R43.2
- new net SH_C: J10.1 (Pin_1), Q3.5, Q3.6, Q3.7, Q3.8, Q3.9, Q5.1, Q5.2, Q5.3, R50.2
- new net SL_C: NT2.2
- new net SN1: NT8.1
- new net SN2: NT6.1
- new net SP1: NT3.1
- new net SP2: NT4.1
Other:
- note added: "Maybe just 100% copy the other phases, just to be safe?"
- note added: "Motor Phases A,B,C"
- note removed: "USE PGO IF I2C PROGRAMMING FAILS"
- moved on the sheet: C53
