File: STM32 - BLDC Driver/DRV8302DCAR.kicad_sch (KiCad schematic)
At the start: 46 parts, among them J3 Conn_01x03_Pin, J5 Conn_01x03_Pin, U3 DRV8302DCAR

Commit message: As manufactured.
Parts:
- removed C17, C37: 0.1uF, symbol Device:C
- removed C18, C20, C21: 100nF, symbol Device:C
- removed C31: 4.7uF, symbol Device:C
- removed R13, R14, R9: 10k, symbol Device:R
- removed R15: 56R, symbol Device:R
- added C11, C12: 4.7u low esr (C1779), Capacitor_SMD:C_0805_2012Metric_Pad1.18x1.45mm_HandSolder, symbol Device:C
- added C33: 0.1uF (C28233), Capacitor_SMD:C_0805_2012Metric_Pad1.18x1.45mm_HandSolder, symbol Device:C
- added C35: 220uF (C46550422), Capacitor_SMD:C_Elec_10x10.2, symbol Device:C
- added C46: 4.7nF (C1744), Capacitor_SMD:C_0805_2012Metric_Pad1.18x1.45mm_HandSolder, symbol Device:C
- added C6: 2.2nF (C28260), Capacitor_SMD:C_0805_2012Metric_Pad1.18x1.45mm_HandSolder, symbol Device:C
- added C7: 1uF (C13832), Capacitor_SMD:C_1206_3216Metric_Pad1.33x1.80mm_HandSolder, symbol Device:C
- added NT1: NetTie_3_Tee, NetTie:NetTie-3_SMD_Pad2.0mm, symbol Device:NetTie_3_Tee
- added R1, R11, R12: 10k (C17414), Resistor_SMD:R_0805_2012Metric_Pad1.20x1.40mm_HandSolder, symbol Device:R
- added R27: 56R (C2930118), Resistor_SMD:R_0603_1608Metric_Pad0.98x0.95mm_HandSolder, symbol Device:R
- C10: renamed from C14; value 120p -> 120p (C107035); footprint (none) -> Capacitor_SMD:C_0603_1608Metric_Pad1.08x0.95mm_HandSolder
- C2: renamed from C24; value 1uF -> 1uF (C13832); footprint (none) -> Capacitor_SMD:C_1206_3216Metric_Pad1.33x1.80mm_HandSolder
- C24: renamed from C33; value 220uF -> 220uF (C46550422); footprint (none) -> Capacitor_SMD:C_Elec_10x10.2
- C25: value 1uF -> 0.1uF (C28233); footprint (none) -> Capacitor_SMD:C_0805_2012Metric_Pad1.18x1.45mm_HandSolder
- C26: value 2.2nF -> 0.1uF (C28233); footprint (none) -> Capacitor_SMD:C_0805_2012Metric_Pad1.18x1.45mm_HandSolder
- C27: renamed from C19; value 47uF_P -> 47uF_P (C18221497); footprint (none) -> Capacitor_SMD:CP_Elec_5x5.4
- C28, C30: value 0.1uF -> 0.1uF (C28233); footprint (none) -> Capacitor_SMD:C_0805_2012Metric_Pad1.18x1.45mm_HandSolder
- C29: value 4.7uF -> 0.1uF (C28233); footprint (none) -> Capacitor_SMD:C_0805_2012Metric_Pad1.18x1.45mm_HandSolder
- C3: renamed from C23; value 2.2uF -> 2.2uF (C920964); footprint (none) -> Capacitor_SMD:C_1206_3216Metric_Pad1.33x1.80mm_HandSolder
- C31: renamed from C35; value 0.1uF -> 0.1uF (C28233); footprint (none) -> Capacitor_SMD:C_0805_2012Metric_Pad1.18x1.45mm_HandSolder
- C32: renamed from C36; value 0.01uF -> 0.01uF (C1710); footprint (none) -> Capacitor_SMD:C_0805_2012Metric_Pad1.18x1.45mm_HandSolder
- C34: value 220uF -> 0.1uF (C28233); footprint (none) -> Capacitor_SMD:C_0805_2012Metric_Pad1.18x1.45mm_HandSolder
- C4: renamed from C16; value 15nF -> 10nF (C1710); footprint (none) -> Capacitor_SMD:C_0805_2012Metric_Pad1.18x1.45mm_HandSolder
- C5: renamed from C27; value 2.2nF -> 2.2nF (C28260); footprint (none) -> Capacitor_SMD:C_0805_2012Metric_Pad1.18x1.45mm_HandSolder
- C8: renamed from C22; value 22nF -> 22nF (C376821); footprint (none) -> Capacitor_SMD:C_0603_1608Metric_Pad1.08x0.95mm_HandSolder
- C9: renamed from C15; value 6.8n -> 6.8n (C1631); footprint (none) -> Capacitor_SMD:C_0603_1608Metric_Pad1.08x0.95mm_HandSolder
- D1: renamed from D4; value D_Zener -> D_Zener (C173406); footprint (none) -> Diode_SMD:D_SOD-123
- D2: renamed from D3; value B330A-13-F -> B330A-13-F (C110485); footprint (none) -> Diode_SMD:D_SMA-SMB_Universal_Handsoldering
- J4: renamed from J3; footprint (none) -> Connector_PinHeader_2.54mm:PinHeader_1x03_P2.54mm_Vertical
- J5: footprint (none) -> Connector_PinHeader_2.54mm:PinHeader_1x03_P2.54mm_Vertical
- L1: renamed from L2; value 22uH -> 22uH (C177244); footprint (none) -> Inductor_SMD:L_Changjiang_FXL0630
- R10: renamed from R18; value 3.3R -> 3.3R (C22979); footprint (none) -> Resistor_SMD:R_0603_1608Metric_Pad0.98x0.95mm_HandSolder
- R13: renamed from R12; value 10k -> 10k (C17414); footprint (none) -> Resistor_SMD:R_0805_2012Metric_Pad1.20x1.40mm_HandSolder
- R18: renamed from R7; value 3k3 -> 3k3 (C22356670); footprint (none) -> Resistor_SMD:R_0603_1608Metric_Pad0.98x0.95mm_HandSolder
- R19: renamed from R6; value 18k -> 18k (C2907111); footprint (none) -> Resistor_SMD:R_0603_1608Metric_Pad0.98x0.95mm_HandSolder
- R2: value 10k -> 10k (C17414); footprint (none) -> Resistor_SMD:R_0805_2012Metric_Pad1.20x1.40mm_HandSolder
- R20: renamed from R5; value 15k -> 15k (C22356635); footprint (none) -> Resistor_SMD:R_0603_1608Metric_Pad0.98x0.95mm_HandSolder
- R26: renamed from R16; value 56R -> 56R (C2930118); footprint (none) -> Resistor_SMD:R_0603_1608Metric_Pad0.98x0.95mm_HandSolder
- R28: renamed from R11; value 1k -> 1k (C22356624); footprint (none) -> Resistor_SMD:R_0603_1608Metric_Pad0.98x0.95mm_HandSolder
- R29: renamed from R10; value 80.6k -> 80.6k (C2960781); footprint (none) -> Resistor_SMD:R_0805_2012Metric_Pad1.20x1.40mm_HandSolder
- R6: renamed from R20; value 4.99k -> 4.99k (C23046); footprint (none) -> Resistor_SMD:R_0603_1608Metric_Pad0.98x0.95mm_HandSolder
- R7: renamed from R4; value 200k -> 200k (C25811); footprint (none) -> Resistor_SMD:R_0603_1608Metric_Pad0.98x0.95mm_HandSolder
- R8: value 1M -> 1M (C26083); footprint (none) -> Resistor_SMD:R_0402_1005Metric_Pad0.72x0.64mm_HandSolder
- R9: renamed from R19; value 34.8k -> 34.8k (C23141); footprint (none) -> Resistor_SMD:R_0603_1608Metric_Pad0.98x0.95mm_HandSolder
- renumbered U3 to U2
Connections:
- net +3V3: now also R11.2, R12.1
- net AGND: now also C7.1, NT1.2; no longer C10.2, C24.1, C25.1, C26.1, C27.2, C28.1, C29.1, C3.1, C30.1, C31.1, C34.1, C4.1, C5.1, C9.2, D2.2 (A), J5.3 (Pin_3), R10.1, R18.1, R2.1, R28.2, R6.1, R7.1, R8.1, U2.57 (PWR_PAD)
- net BST_A: now also C25.2
- net BST_B: now also C26.2
- net BST_C: now also C28.2
- net DRV_BST_BK: now also C34.2
- net DVDD: now also C7.2; no longer C25.2
- net GAIN: now also R1.2; no longer R2.2
- net PVDD: now also C29.2, C30.2, U2.29 (PVDD1), U2.53 (PVDD2), U2.54 (PVDD2), C11.1, C12.1, C35.2; no longer C34.2
- net PVDDSENSE: now also C33.2
- net SH_A: now also C25.1
- net SH_B: now also C26.1
- net SH_C: now also C28.1
- net SO1: now also C6.2, R27.2; no longer C26.2
- net nFAULT: now also R11.1
- net nOCTW: now also R12.2
- net at C4.2, U2.56 (SS_TR): now also C46.2
- net at D2.1 (K), L1.1, U2.50 (PH)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: now also C34.1
- net at U2.25 (SO1): now also R27.1
- net OC_ADJ: now reaches J4.2 (Pin_2), U2.11 (OC_ADJ)
- net at U2.7 (DTC): now also R2.2
- removed net +24V: C28.2, C29.2, C30.2, U2.29 (PVDD1), U2.53 (PVDD2), U2.54 (PVDD2)
- new net GND: C10.2, C11.2, C12.2, C27.2, C29.1, C3.1, C30.1, C33.1, C4.1, C46.1, C5.1, C6.1, C9.2, D2.2 (A), J5.3 (Pin_3), NT1.1, R1.1, R18.1, R2.1, R28.2, R6.1, R7.1, R8.1, U2.57 (PWR_PAD)
- new net PGND: C24.1, C31.1, C35.1, NT1.3, R10.1
