File: STM32 - BLDC Driver/STM32G.kicad_sch (KiCad schematic)
At the start: 39 parts, among them J2 Conn_01x03_Pin, J4 TC2050, J6 Conn_01x04_Pin, J7 FH34SRJ-10S-0.5SH_50_, J8 Conn_01x03_Pin, P1 USB_C_Plug_USB2.0, U1 STM32F411CEUx, U6 LD1117S33TR_SOT223, U8 LM66100DCK, Y1 Crystal_GND24

Commit message: As manufactured.
Parts:
- removed C10: 4.7u low esr, symbol Device:C
- removed C11, C12, C4, C5, C6, C7, C8: 100n, symbol Device:C
- removed C46: 100nF, symbol Device:C
- removed P1: USB_C_Plug_USB2.0, symbol Connector:USB_C_Plug_USB2.0
- removed R36, R37: 22R, symbol Device:R
- removed R38: 5.1k, symbol Device:R
- removed R40: 5Ohm, symbol Device:R
- removed R42: 2.2k, symbol Device:R
- removed R43: 10k, symbol Device:R
- removed TP23, TP24, TP25, TP26, TP27, TP28, TP29, TP30, TP31: TestPoint, symbol Connector:TestPoint
- removed U8: LM66100DCK, Package_TO_SOT_SMD:SOT-363_SC-70-6, symbol Power_Management:LM66100DCK
- added C1: 4.7u low esr (C1779), Capacitor_SMD:C_0805_2012Metric_Pad1.18x1.45mm_HandSolder, symbol Device:C
- added C14, C15, C16, C18, C19, C21, C22, C23: 100nF 50V (C28233), Capacitor_SMD:C_0805_2012Metric_Pad1.18x1.45mm_HandSolder, symbol Device:C
- added H1, H2, H3, H4: MountingHole_Pad, MountingHole:MountingHole_3.2mm_M3_Pad_Via, symbol Mechanical:MountingHole_Pad
- added J8: GT-USB-7010B, GT-USB-7010B:G-SWITCH_GT-USB-7010B, symbol GT-USB-7010B:GT-USB-7010B
- added NT5: NetTie_2, NetTie:NetTie-2_SMD_Pad0.5mm, symbol Device:NetTie_2
- added R14, R15: 5.1k (C22356620), Resistor_SMD:R_0603_1608Metric_Pad0.98x0.95mm_HandSolder, symbol Device:R
- added R16, R17: 0R, Resistor_SMD:R_0603_1608Metric_Pad0.98x0.95mm_HandSolder, symbol Device:R
- added R23: 2.2k (C4190), Resistor_SMD:R_0603_1608Metric_Pad0.98x0.95mm_HandSolder, symbol Device:R
- added R5: 10k (C17414), Resistor_SMD:R_0805_2012Metric_Pad1.20x1.40mm_HandSolder, symbol Device:R
- added TP6: TestPoint, TestPoint:TestPoint_Pad_D4.0mm, symbol Connector:TestPoint
- C13: value 100n -> 100nF 50V (C28233); footprint (none) -> Capacitor_SMD:C_0805_2012Metric_Pad1.18x1.45mm_HandSolder
- C17: renamed from C9; value 2.2u -> 2.2u C5448893; footprint (none) -> Capacitor_SMD:C_0805_2012Metric_Pad1.18x1.45mm_HandSolder
- C20: renamed from C47; value 10uF -> 10uF (C15850); footprint (none) -> Capacitor_SMD:C_0805_2012Metric_Pad1.18x1.45mm_HandSolder
- J1: renamed from J7; footprint FH34SRJ-10S-0.5SH_50_:HRS_FH34SRJ-10S-0.5SH_50_ -> FH34SRJ-10S-0.5SH:HRS_FH34SRJ-10S-0.5SH_50_
- J2: renamed from J8; footprint (none) -> Connector_PinHeader_2.54mm:PinHeader_1x03_P2.54mm_Vertical
- J3: renamed from J6; footprint (none) -> Connector_PinHeader_2.54mm:PinHeader_1x04_P2.54mm_Vertical
- J7: renamed from J2; footprint (none) -> Connector_PinHeader_2.54mm:PinHeader_1x03_P2.54mm_Vertical
- R21: renamed from R41; value 2.2k -> 2.2k (C4190); footprint (none) -> Resistor_SMD:R_0603_1608Metric_Pad0.98x0.95mm_HandSolder
- R4: renamed from R3; value 0R -> 0R (C17477); footprint (none) -> Resistor_SMD:R_0805_2012Metric_Pad1.20x1.40mm_HandSolder
- Y1: value Crystal_GND24 -> Crystal_GND24 (C5444547); footprint (none) -> Crystal:Crystal_SMD_3225-4Pin_3.2x2.5mm_HandSoldering
- renumbered J4 to J6, U6 to U4, U1 to U5
Connections:
- net +3V3: now also C13.2, C14.2, C15.2, C16.2, C22.2, NT5.1, R23.2, R5.2; no longer J1.1
- net AS5600_SDA: now also R23.1
- net GND: now also C13.1, J2.3 (Pin_3), C1.2, C14.1, C15.1, C16.1, C18.2, C19.1, C21.1, C22.1, C23.1, H1.1, H2.1, H3.1, H4.1, J8.A1_B12 (GND_A), J8.B1_A12 (GND_B), J8.SH1 (SHIELD), J8.SH2 (SHIELD), J8.SH3 (SHIELD), J8.SH4 (SHIELD), R14.2, R15.2; no longer C13.2
- net HALL_A: now also U5.41 (PB5); no longer U5.40 (PB4)
- net HALL_B: now also U5.40 (PB4); no longer U5.41 (PB5)
- net MCU_NRST: now also C18.1; no longer J2.3 (Pin_3)
- net MCU_OSC_IN: now also C21.2; no longer C13.1
- net MCU_VCAP1: now also C1.1
- net NTC_2: now also TP6.1
- net STM_D+: now also R17.2
- net STM_D-: now also R16.2
- net USB_VBUS: now also C23.2, J8.A4_B9 (VBUS_A), J8.B4_A9 (VBUS_B)
- net XTA_IN: now also C19.2
- net at J2.1 (Pin_1): now also R5.1
- net USB_3V3: now reaches C20.1, U4.2 (VO)
- net AS5600_OUT: no longer names the net of U5.3 (PC14)
- new net: J8.A5 (CC1), R15.1
- new net: J8.B5 (CC2), R14.1
- new net 5V: J1.1
- new net D+: J8.A6 (D1+), J8.B7 (D2-), R17.1
- new net D-: J8.A7 (D1-), J8.B6 (D2+), R16.1
- new net DRV8302_REF: NT5.2
- no-connect marks 7 -> 9
Other:
- note removed: "This should prevent reverse current"
