File: STM32 - BLDC Driver/Sensors.kicad_sch (KiCad schematic)
At the start: 6 parts, among them U5 BMI088 (C194919)

Commit message: As manufactured.
Parts:
- removed C44, C45: 100nF (C1711), Capacitor_SMD:C_0805_2012Metric_Pad1.18x1.45mm_HandSolder, symbol Device:C
- removed TP20: TestPoint, symbol Connector:TestPoint
- removed U5: BMI088 (C194919), BMI088:PQFN50P450X300X100-16N, symbol BMI088:BMI088
- added TP10: TestPoint, TestPoint:TestPoint_Pad_D3.0mm, symbol Connector:TestPoint
- R31: renamed from R33; value R -> 8.2k (C17828); footprint (none) -> Resistor_SMD:R_0805_2012Metric_Pad1.20x1.40mm_HandSolder
Connections:
- net MOS1_NTC: now also TP10.1
- no-connect marks 1 -> 0
